Commit message: many changes

File: fyp_ws/src/drift_car_description/urdf/drift_car.urdf.xacro (robot description, xacro)
@@ -236,5 +236,5 @@
   </link>
   <gazebo reference="base_link">
-    <material>Gazebo/Grey</material>
+    <material>Gazebo/Red</material>
   </gazebo>
   <joint name="imu_joint" type="fixed">
@@ -285,5 +285,5 @@
   </link>
   <gazebo reference="chassis">
-    <material>Gazebo/Grey</material>
+    <material>Gazebo/Red</material>
   </gazebo>
   <joint name="base_link_to_chasis" type="fixed">
